File: hardware/NixiePower.brd (EAGLE design)
At the start: 33.5 x 36 mm, 25 parts, among them IC1 TJ34063A, T1 R6006AND

Commit message: Update BOM
Parts:
- C11: value (none) -> 4.7µ
- R1: value (none) -> 10k
- R12: value 30k -> 6k
- R9: value 4.7M -> 1M
Changed lines of the file:
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@@
 <grid distance="50" unitdist="mil" unit="mm" style="dots" multiple="1" display="yes" altdistance="5" altunitdist="mil" altunit="mm"/>
 <layers>
-<layer number="1" name="Top" color="4" fill="1" visible="yes" active="yes"/>
+<layer number="1" name="Top" color="4" fill="1" visible="no" active="yes"/>
 <layer number="2" name="Route2" color="16" fill="1" visible="no" active="no"/>
 <layer number="3" name="Route3" color="17" fill="1" visible="no" active="no"/>
@@
 <layer number="19" name="Unrouted" color="6" fill="1" visible="yes" active="yes"/>
 <layer number="20" name="Dimension" color="24" fill="1" visible="yes" active="yes"/>
-<layer number="21" name="tPlace" color="7" fill="1" visible="yes" active="yes"/>
+<layer number="21" name="tPlace" color="7" fill="1" visible="no" active="yes"/>
 <layer number="22" name="bPlace" color="7" fill="1" visible="yes" active="yes"/>
-<layer number="23" name="tOrigins" color="15" fill="1" visible="yes" active="yes"/>
+<layer number="23" name="tOrigins" color="15" fill="1" visible="no" active="yes"/>
 <layer number="24" name="bOrigins" color="15" fill="1" visible="yes" active="yes"/>
-<layer number="25" name="tNames" color="7" fill="1" visible="yes" active="yes"/>
+<layer number="25" name="tNames" color="7" fill="1" visible="no" active="yes"/>
 <layer number="26" name="bNames" color="7" fill="1" visible="yes" active="yes"/>
 <layer number="27" name="tValues" color="7" fill="1" visible="no" active="yes"/>
@@
 <layer number="37" name="tTest" color="7" fill="1" visible="no" active="yes"/>
 <layer number="38" name="bTest" color="7" fill="1" visible="no" active="yes"/>
-<layer number="39" name="tKeepout" color="4" fill="11" visible="yes" active="yes"/>
+<layer number="39" name="tKeepout" color="4" fill="11" visible="no" active="yes"/>
 <layer number="40" name="bKeepout" color="1" fill="11" visible="yes" active="yes"/>
-<layer number="41" name="tRestrict" color="4" fill="10" visible="yes" active="yes"/>
+<layer number="41" name="tRestrict" color="4" fill="10" visible="no" active="yes"/>
 <layer number="42" name="bRestrict" color="1" fill="10" visible="yes" active="yes"/>
 <layer number="43" name="vRestrict" color="2" fill="10" visible="no" active="yes"/>
@@
 <layer number="49" name="Reference" color="7" fill="1" visible="no" active="yes"/>
 <layer number="50" name="dxf" color="7" fill="1" visible="no" active="no"/>
-<layer number="51" name="tDocu" color="7" fill="1" visible="yes" active="yes"/>
+<layer number="51" name="tDocu" color="7" fill="1" visible="no" active="yes"/>
 <layer number="52" name="bDocu" color="7" fill="1" visible="yes" active="yes"/>
 <layer number="88" name="SimResults" color="9" fill="1" visible="no" active="no"/>
@@
 </element>
 <element name="T1" library="mosfets" package="CPT3" value="R6006AND" x="-11.43" y="1.27" smashed="yes" rot="MR180"/>
-<element name="R9" library="rcl" library_urn="urn:adsk.eagle:library:334" package="R0603" package3d_urn="urn:adsk.eagle:package:23555/3" value="4.7M" x="0" y="-12.7" smashed="yes" rot="MR180">
+<element name="R9" library="rcl" library_urn="urn:adsk.eagle:library:334" package="R0603" package3d_urn="urn:adsk.eagle:package:23555/3" value="1M" x="0" y="-12.7" smashed="yes" rot="MR180">
 <attribute name="NAME" x="2.286" y="-12.7" size="0.8128" layer="26" font="vector" rot="MR90" align="center"/>
 <attribute name="POPULARITY" value="77" x="0" y="-12.7" size="1.778" layer="28" rot="MR180" display="off"/>
@@
 <attribute name="VALUE" x="-0.635" y="-10.795" size="1.27" layer="28" rot="MR180"/>
 </element>
-<element name="R12" library="rcl" library_urn="urn:adsk.eagle:library:334" package="R0603" package3d_urn="urn:adsk.eagle:package:23555/3" value="30k" x="0" y="-10.668" smashed="yes" rot="MR180">
+<element name="R12" library="rcl" library_urn="urn:adsk.eagle:library:334" package="R0603" package3d_urn="urn:adsk.eagle:package:23555/3" value="6k" x="0" y="-10.668" smashed="yes" rot="MR180">
 <attribute name="NAME" x="2.286" y="-10.668" size="0.8128" layer="26" font="vector" rot="MR90" align="center"/>
 <attribute name="POPULARITY" value="77" x="0" y="-10.668" size="1.778" layer="28" rot="MR180" display="off"/>
@@
 <attribute name="SPICEPREFIX" value="C" x="0" y="-8.255" size="1.778" layer="28" rot="MR0" display="off"/>
 </element>
-<element name="C11" library="rcl" library_urn="urn:adsk.eagle:library:334" package="E5-10,5" package3d_urn="urn:adsk.eagle:package:23372/2" value="" x="11.43" y="-11.43" smashed="yes">
+<element name="C11" library="rcl" library_urn="urn:adsk.eagle:library:334" package="E5-10,5" package3d_urn="urn:adsk.eagle:package:23372/2" value="4.7µ" x="11.43" y="-11.43" smashed="yes">
 <attribute name="NAME" x="11.43" y="-14.0208" size="0.8128" layer="25" font="vector" ratio="10" align="center"/>
 <attribute name="POPULARITY" value="23" x="11.43" y="-11.43" size="1.778" layer="27" display="off"/>
@@
 <attribute name="VALUE" x="14.605" y="3.175" size="1.27" layer="28" rot="MR0"/>
 </element>
-<element name="R1" library="rcl" library_urn="urn:adsk.eagle:library:334" package="R0603" package3d_urn="urn:adsk.eagle:package:23555/3" value="" x="2.54" y="7.62" smashed="yes" rot="MR270">
+<element name="R1" library="rcl" library_urn="urn:adsk.eagle:library:334" package="R0603" package3d_urn="urn:adsk.eagle:package:23555/3" value="10k" x="2.54" y="7.62" smashed="yes" rot="MR270">
 <attribute name="NAME" x="3.81" y="7.62" size="0.8128" layer="26" font="vector" rot="MR270" align="center"/>
 <attribute name="POPULARITY" value="77" x="2.54" y="7.62" size="1.778" layer="28" rot="MR270" display="off"/>
